Commit message: added lidar and camera to .xacro file

File: src/my_robot/urdf/my_robot.xacro (robot description, xacro)
@@ -121,3 +121,65 @@
      <dynamics damping="1.0" friction="1.0"/>
    </joint>
+   <!-- camera -->
+   <link name="camera">
+   	<inertial>
+   		<mass value="0.1"/>
+   		<origin xyz="0 0 0" rpy="0 0 0"/>
+   		<inertia
+   			ixx="1e-6" ixy="0" ixz="0"
+   			iyy="1e-6" iyz="0"
+   			izz="1e-6"
+   		/>
+   	</inertial>
+   	<collision name="camera_collision">
+   		<origin xyz="0 0 0" rpy="0 0 0"/>
+   		<geometry>
+   			<box size="0.05 0.05 0.05"/>
+   		</geometry>
+   	</collision>
+   	<visual name="camera_visual">
+   		<origin xyz="0 0 0" rpy="0 0 0"/>
+   		<geometry>
+   			<box size="0.05 0.05 0.05"/>
+   		</geometry>
+   	</visual>
+   </link>
+   <!-- camera joint -->
+   <joint type="fixed" name="camera_joint">
+   	<origin xyz="0.2 0 0" rpy="0 0 0"/>
+   	<child link="camera"/>
+   	<parent link="chassis"/>
+   	<axis xyz="0 1 0" rpy="0 0 0"/>
+   </joint>
+   <!-- lidar -->
+   <link name="hokuyo">
+   	<inertial>
+   		<mass value="1e-5"/>
+   		<origin xyz="0 0 0" rpy="0 0 0"/>
+   		<inertia
+        ixx="1e-6" ixy="0" ixz="0"
+        iyy="1e-6" iyz="0"
+        izz="1e-6"
+      />
+   	</inertial>
+   	<collision name="hokuyo_collision">
+   		<origin xyz="0 0 0" rpy="0 0 0"/>
+   		<geometry>
+   			<box size="0.1 0.1 0.1"/>
+   		</geometry>
+   	</collision>
+   	<visual name="hokuyo_visual">
+   		<origin xyz="0 0 0" rpy="0 0 0"/>
+   		<geometry>
+   			<mesh filename="package://my_robot/meshes/hokuyo.dae"/>
+   		</geometry>
+   	</visual>
+   </link>
+   <!-- lidar joint -->
+   <joint type="fixed" name="hokuyo_joint">
+   	<origin xyz="0.15 0 0.1" rpy="0 0 0"/>
+   	<child link="hokuyo"/>
+   	<parent link="chassis"/>
+   	<axis xyz="0 1 0" rpy="0 0 0"/>
+   </joint>
 </robot>

Commit message: finished rviz integration

File: src/my_robot/urdf/my_robot.xacro (robot description, xacro)
@@ -1,4 +1,5 @@
 <?xml version='1.0'?>
 <robot name="my_robot" xmlns:xacro="http://www.ros.org/wiki/xacro">
+  <xacro:include filename="$(find my_robot)/urdf/my_robot.gazebo" />
   <link name="robot_footprint"></link>
   <joint name="robot_footprint_joint" type="fixed">
@@ -88,4 +89,7 @@
      <dynamics damping="1.0" friction="1.0"/>
    </joint>
+   <gazebo reference="left_wheel">
+      <material>Gazebo/Black</material>
+   </gazebo>
   <!-- right wheel linke -->
   <link name="right_wheel">
@@ -121,4 +125,7 @@
      <dynamics damping="1.0" friction="1.0"/>
    </joint>
+   <gazebo reference="right_wheel">
+      <material>Gazebo/Black</material>
+   </gazebo>
    <!-- camera -->
    <link name="camera">
@@ -152,4 +159,7 @@
    	<axis xyz="0 1 0" rpy="0 0 0"/>
    </joint>
+   <gazebo reference="camera">
+      <material>Gazebo/Black</material>
+   </gazebo>
    <!-- lidar -->
    <link name="hokuyo">
@@ -183,3 +193,6 @@
    	<axis xyz="0 1 0" rpy="0 0 0"/>
    </joint>
+   <gazebo reference="hokuyo">
+      <material>Gazebo/Black</material>
+   </gazebo>
 </robot>
